Commit message: PR2: tight re-spherization of base/torso/forearm/wrist/palm (124->312 spheres)
The original 8-sphere base and torso covers overshot the real geometry by
~10cm laterally (base spheres also poked 6cm below ground), and the 6-sphere
forearm by ~2.6cm. Reaching over a table, 62% of all VAMP conf rejections
were false positives against the table (probe vs the GJK oracle), inflating
the stance-solver re-fan rate 4x on pr2_anomaly.

New covers: base slab-decomposed into column grids (61 spheres, <=3.5cm
lateral, bottoms clipped to ground tangency per the spot/fetchx convention),
torso 63, and hull set-covers at 1cm grow-margin for forearm (30), wrist
flex (10), gripper palm (12) per arm. SRDF gains the adjacent pairs the
denser covers now touch at the tucked conf (torso~head_tilt,
forearm~own-gripper fingers).

False positives 6849 -> 2353 (remainder is sub-12mm-clearance confs, below
spherization resolution); pr2_anomaly e2e 40-51 s/goal -> 13.7 s/goal,
passes in 7.8 min with zero bogus kin-exhausted verdicts.

Co-Authored-By: Claude Fable 5 <noreply@anthropic.com>

File: resources/pr2/pr2x_spherized.urdf (robot description, URDF)
Before this commit: robot pr2, 38 links, 37 joints
Links:
- link base_link: geometry collision sphere radius=0.0750; collision sphere radius=0.0750
- link l_forearm_link: geometry collision sphere radius=0.0353; collision sphere radius=0.0361
- link l_gripper_palm_link: geometry collision sphere radius=0.0281; collision sphere radius=0.0281
- link l_wrist_flex_link: geometry collision sphere radius=0.0223; collision sphere radius=0.0223
- link r_forearm_link: geometry collision sphere radius=0.0353; collision sphere radius=0.0361
- link r_gripper_palm_link: geometry collision sphere radius=0.0281; collision sphere radius=0.0281
- link r_wrist_flex_link: geometry collision sphere radius=0.0223; collision sphere radius=0.0223
- link torso_lift_link: geometry collision sphere radius=0.0735; collision sphere radius=0.0735
