Commit message: Rainbow: split into Rainbow (ZED+lidar) and RainbowCam (+wrist cameras)
Two cricket-input model sets sharing all kinematics:
  * rainbow_spherized*     -- base Rainbow: 197 spheres (196 + ZED head sphere).
                              The lidar is exact-model only (inert in spheres).
  * rainbowcam_spherized*  -- RainbowCam: 199 spheres (+2 wrist-camera spheres),
                              generated as base + a wrist fragment.
  * rainbowcam{,l}.json    -- fkcc_gen configs for the RainbowCam header pair.

The wrist cameras are the ONLY difference; ZED and lidar are on both.

Co-Authored-By: Claude Opus 4.8 <noreply@anthropic.com>

File: resources/rainbow/rainbowcam_spherized.urdf (robot description, URDF)
Before this commit: robot RB_Y1_V1.0.1, 40 links, 39 joints
Links:
- added link link_left_arm_camera; collision sphere radius=0.04668
- added link link_right_arm_camera; collision sphere radius=0.04668
Joints:
- added joint left_arm_camera_mount: type fixed, parent FT_sensor_L, child link_left_arm_camera, origin xyz=0 0 0 rpy=0 0 0
- added joint right_arm_camera_mount: type fixed, parent FT_sensor_R, child link_right_arm_camera, origin xyz=0 0 0 rpy=0 0 0
