Commit message: Clip spot/fetchx base spheres to the ground plane
Companion to vamp: spheres on base-fixed links whose bottoms fell below
the standing plane (spot body/payload: 20, fetch base_link: 3) are
clipped to bottom-tangency. Floor-welded HPN problems made every conf
collide otherwise; rainbow already respects the z>=0 convention.

Co-Authored-By: Claude Fable 5 <noreply@anthropic.com>

File: resources/fetch/fetchx_spherized.urdf (robot description, URDF)
Before this commit: robot fetch, 21 links, 20 joints
Links:
- link base_link: geometry collision sphere radius=0.066; collision sphere radius=0.066

File: resources/spot/spotx_spherized.urdf (robot description, URDF)
Before this commit: robot spot, 17 links, 16 joints
Links:
- link body: geometry collision sphere radius=0.056700; collision sphere radius=0.062000

Commit message: Point the VAMP end effectors at the standard TCP frame
Regeneration inputs for vamp@031d5c59 (see
../HPN/docs/gripper_frame_standardization.md): each spherized URDF gains the
standard TCP frame as a fixed joint off its existing end frame, and each config's
end_effector names it -- fetch_rarm_tcp / r_gripper_tcp / tcp_right / tcp_left /
arm_tcp. Attachment transforms are expressed in that frame, so the compiled FK
has to know it.

Regenerated .hh sphere counts are unchanged (111/312/197/199/108), which is the
check that matters: a collapse there would mean the SRDF comment trap.

movo is patched the same way but its resources are untracked in this repo, so
its regeneration is not captured here.

Co-Authored-By: Claude Opus 5 <noreply@anthropic.com>

File: resources/fetch/fetchx_spherized.urdf (robot description, URDF)
Before this commit: robot fetch, 21 links, 20 joints
Links:
- added link fetch_rarm_tcp
Joints:
- added joint fetch_rarm_tcp_joint: type fixed, parent fetch_rarm_end, child fetch_rarm_tcp, origin xyz=0 0 0 rpy=-3.14159265358979 0 1.57079632679490

File: resources/pr2/pr2x_spherized.urdf (robot description, URDF)
Before this commit: robot pr2, 38 links, 37 joints
Links:
- added link r_gripper_tcp
Joints:
- added joint r_gripper_tcp_joint: type fixed, parent r_gripper_tool_frame, child r_gripper_tcp, origin xyz=0.006 0 0 rpy=1.57079632679490 0 1.57079632679490

File: resources/rainbow/rainbow_spherized_plus.urdf (robot description, URDF)
Before this commit: robot RB_Y1_V1.0.1, 40 links, 39 joints
Links:
- added link tcp_left
- added link tcp_right
Joints:
- added joint tcp_joint_left: type fixed, parent grasp_frame_left, child tcp_left, origin xyz=0 0 0 rpy=-3.14159265358979 0 1.57079632679490
- added joint tcp_joint_right: type fixed, parent grasp_frame_right, child tcp_right, origin xyz=0 0 0 rpy=-3.14159265358979 0 1.57079632679490

File: resources/rainbow/rainbowcam_spherized_plus.urdf (robot description, URDF)
Before this commit: robot RB_Y1_V1.0.1, 42 links, 41 joints
Links:
- added link tcp_left
- added link tcp_right
Joints:
- added joint tcp_joint_left: type fixed, parent grasp_frame_left, child tcp_left, origin xyz=0 0 0 rpy=-3.14159265358979 0 1.57079632679490
- added joint tcp_joint_right: type fixed, parent grasp_frame_right, child tcp_right, origin xyz=0 0 0 rpy=-3.14159265358979 0 1.57079632679490

File: resources/spot/spotx_spherized.urdf (robot description, URDF)
Before this commit: robot spot, 17 links, 16 joints
Links:
- added link arm_tcp
Joints:
- added joint arm_tcp_joint: type fixed, parent arm_end_effector_link, child arm_tcp, origin xyz=0 0 0 rpy=-3.14159265358979 0 1.57079632679490
