Commit message: Droid: spheres over the full joint ranges, base above the floor, camera with its bracket clamp
resources/droid: the inputs of vamp's droid kernel, 458 spheres.
- Over the master's full joint ranges; the joint-6 limit of d517caf is gone,
  so link5-link7, link5-wrist_camera and link2-link6 are all checked.
- Base spheres stay above the base plane (bottoms at z >= 0.5 mm, covering
  the hull from z = 12 mm up). Reaching z = -0.015 collided with the PO
  worlds' permanent floor body at every conf (vamp 1ba2916, reverted).
- The camera's spheres cover the master's new camera hull, which now
  includes the DROID bracket's side clamp (QAA 9204987); only
  wrist_camera_link was re-covered.

tools/spherize: respherize.py floors the base above z = 0; mix_urdf.py
splices one model's link spheres into another (the camera re-cover, and
bisecting a kernel regression). README: both recipes and the audits.

Co-Authored-By: Claude Opus 5.5 <noreply@anthropic.com>

File: resources/droid/droid_spherized.urdf (robot description, URDF)
Before this commit: robot droid, 42 links, 41 joints
Links:
- link panda_link0: geometry collision sphere radius=0.024891; collision sphere radius=0.025717
- link panda_link0__s1: geometry collision sphere radius=0.010000; collision sphere radius=0.018194
- link panda_link0__s2: geometry collision sphere radius=0.010048; collision sphere radius=0.017338
- link wrist_camera_link: geometry collision sphere radius=0.012040; collision sphere radius=0.016092
- link wrist_camera_link__s1: geometry collision sphere radius=0.012011; collision sphere radius=0.012023
- link wrist_camera_link__s2: geometry collision sphere radius=0.015977; collision sphere radius=0.016009
- link wrist_camera_link__s3: geometry collision sphere radius=0.011909; collision sphere radius=0.011944
Joints:
- joint panda_joint6: limit lower=0.95 upper=4.5169 effort=12.0 velocity=4.18 -> lower=0.5445 upper=4.5169 effort=12.0 velocity=4.18
